File: reTerminalEM-NVMe-mPCIe-USB/reTerminalEM-NVMe-mPCIe-USB.kicad_pcb (KiCad board)
At the start: 2 copper layers, 135 x 90.4 mm, 65 parts, among them J1 FX23-100S-0.5SV, J10 USB1, J11 HD1, J12 HD2, J13 HD3, J14 HD4, J2 M.2, J3 J_Standoff_M3_H2.5, J4 mPCIe, J5 J_SIM_Card_Nano_6P_Shielded, J6 J_Standoff_M3_H2.5, J7 J_Standoff_M3_H2.5, U4 USB2514B, Y3 24MHz

Commit message: no message
Parts:
- J2: value M.2 -> 1-2199230-5
- J6, J7: value J_Standoff_M3_H2.5 -> J_Standoff_M2_H4; footprint StanleyProjects:WE_WA-SMSI_9774025360 -> StanleyProjects:WE_WA-SMSI_9774040243
Connections:
- C33 pad 1: 3V3_PCI -> unconnected-(C33-Pad1)
- C33 pad 2: GND -> unconnected-(C33-Pad2)
- C35 pad 1: 3V3_PCI -> unconnected-(C35-Pad1)
- C35 pad 2: GND -> unconnected-(C35-Pad2)
- J1 pad 28: Net-(J1-Pad28) -> unconnected-(J1-Pad28)
- J1 pad 30: Net-(J1-Pad30) -> unconnected-(J1-Pad30)
- J1 pad 34: Net-(J1-Pad34) -> unconnected-(J1-Pad34)
- J1 pad 36: Net-(J1-Pad36) -> unconnected-(J1-Pad36)
- J1 pad 37: Net-(J1-Pad37) -> unconnected-(J1-Pad37)
- J1 pad 39: Net-(J1-Pad39) -> unconnected-(J1-Pad39)
- J1 pad 40: Net-(J1-Pad40) -> unconnected-(J1-Pad40)
- J1 pad 41: Net-(J1-Pad41) -> unconnected-(J1-Pad41)
- J1 pad 42: Net-(J1-Pad42) -> unconnected-(J1-Pad42)
- J1 pad 43: Net-(J1-Pad43) -> unconnected-(J1-Pad43)
- J1 pad 46: Net-(J1-Pad46) -> unconnected-(J1-Pad46)
- J1 pad 48: Net-(J1-Pad48) -> unconnected-(J1-Pad48)
- J1 pad 49: Net-(J1-Pad49) -> unconnected-(J1-Pad49)
- J1 pad 51: Net-(J1-Pad51) -> unconnected-(J1-Pad51)
- J1 pad 64: Net-(J1-Pad64) -> unconnected-(J1-Pad64)
- J1 pad 66: Net-(J1-Pad66) -> unconnected-(J1-Pad66)
- J1 pad 70: Net-(J1-Pad70) -> unconnected-(J1-Pad70)
- J1 pad 72: Net-(J1-Pad72) -> unconnected-(J1-Pad72)
- J1 pad 78: Net-(J1-Pad78) -> unconnected-(J1-Pad78)
- J1 pad 80: Net-(J1-Pad80) -> unconnected-(J1-Pad80)
- J1 pad 81: Net-(J1-Pad81) -> unconnected-(J1-Pad81)
- J1 pad 82: Net-(J1-Pad82) -> unconnected-(J1-Pad82)
- J1 pad 83: Net-(J1-Pad83) -> unconnected-(J1-Pad83)
- J1 pad 84: Net-(J1-Pad84) -> unconnected-(J1-Pad84)
- J1 pad 85: Net-(J1-Pad85) -> unconnected-(J1-Pad85)
- J1 pad 86: Net-(J1-Pad86) -> unconnected-(J1-Pad86)
- J1 pad 87: Net-(J1-Pad87) -> unconnected-(J1-Pad87)
- J1 pad 89: Net-(J1-Pad89) -> unconnected-(J1-Pad89)
- J1 pad 90: Net-(J1-Pad90) -> unconnected-(J1-Pad90)
- J1 pad 91: Net-(J1-Pad91) -> unconnected-(J1-Pad91)
- J1 pad 93: Net-(J1-Pad93) -> unconnected-(J1-Pad93)
- J1 pad 94: Net-(J1-Pad94) -> unconnected-(J1-Pad94)
- J1 pad 95: Net-(J1-Pad95) -> unconnected-(J1-Pad95)
- J1 pad 97: Net-(J1-Pad97) -> unconnected-(J1-Pad97)
- J1 pad 98: Net-(J1-Pad98) -> unconnected-(J1-Pad98)
- J1 pad MH2: GND -> unconnected-(J1-PadMH2)
- J1 pad MH3: GND -> unconnected-(J1-PadMH3)
- J2 pad 11: Net-(J2-Pad11) -> unconnected-(J2-Pad11)
- J2 pad 13: Net-(J2-Pad13) -> unconnected-(J2-Pad13)
- J2 pad 17: Net-(J2-Pad17) -> unconnected-(J2-Pad17)
- J2 pad 19: Net-(J2-Pad19) -> unconnected-(J2-Pad19)
- J2 pad 20: Net-(J2-Pad20) -> unconnected-(J2-Pad20)
- J2 pad 22: Net-(J2-Pad22) -> unconnected-(J2-Pad22)
- J2 pad 23: Net-(J2-Pad23) -> unconnected-(J2-Pad23)
- J2 pad 24: Net-(J2-Pad24) -> unconnected-(J2-Pad24)
- J2 pad 25: Net-(J2-Pad25) -> unconnected-(J2-Pad25)
- J2 pad 26: Net-(J2-Pad26) -> unconnected-(J2-Pad26)
- J2 pad 28: Net-(J2-Pad28) -> unconnected-(J2-Pad28)
- J2 pad 29: Net-(J2-Pad29) -> unconnected-(J2-Pad29)
- J2 pad 30: Net-(J2-Pad30) -> unconnected-(J2-Pad30)
- J2 pad 31: Net-(J2-Pad31) -> unconnected-(J2-Pad31)
- J2 pad 32: Net-(J2-Pad32) -> unconnected-(J2-Pad32)
- J2 pad 34: Net-(J2-Pad34) -> unconnected-(J2-Pad34)
- J2 pad 35: Net-(J2-Pad35) -> unconnected-(J2-Pad35)
- J2 pad 36: Net-(J2-Pad36) -> unconnected-(J2-Pad36)
- J2 pad 37: Net-(J2-Pad37) -> unconnected-(J2-Pad37)
- J2 pad 40: Net-(J2-Pad40) -> unconnected-(J2-Pad40)
- J2 pad 42: Net-(J2-Pad42) -> unconnected-(J2-Pad42)
- J2 pad 44: Net-(J2-Pad44) -> unconnected-(J2-Pad44)
- J2 pad 46: Net-(J2-Pad46) -> unconnected-(J2-Pad46)
- J2 pad 48: Net-(J2-Pad48) -> unconnected-(J2-Pad48)
- J2 pad 5: Net-(J2-Pad5) -> unconnected-(J2-Pad5)
- J2 pad 56: Net-(J2-Pad56) -> unconnected-(J2-Pad56)
- J2 pad 58: Net-(J2-Pad58) -> unconnected-(J2-Pad58)
- J2 pad 6: Net-(J2-Pad6) -> unconnected-(J2-Pad6)
- J2 pad 67: Net-(J2-Pad67) -> unconnected-(J2-Pad67)
- J2 pad 68: Net-(J2-Pad68) -> unconnected-(J2-Pad68)
- J2 pad 69: Net-(J2-Pad69) -> unconnected-(J2-Pad69)
- J2 pad 7: Net-(J2-Pad7) -> unconnected-(J2-Pad7)
- J2 pad 8: Net-(J2-Pad8) -> unconnected-(J2-Pad8)
- J4 pad 1: Net-(J4-Pad1) -> unconnected-(J4-Pad1)
- J4 pad 11: Net-(J4-Pad11) -> unconnected-(J4-Pad11)
- J4 pad 13: Net-(J4-Pad13) -> unconnected-(J4-Pad13)
- J4 pad 17: Net-(J4-Pad17) -> unconnected-(J4-Pad17)
- J4 pad 19: Net-(J4-Pad19) -> unconnected-(J4-Pad19)
- J4 pad 20: Net-(J4-Pad20) -> unconnected-(J4-Pad20)
- J4 pad 22: Net-(J4-Pad22) -> unconnected-(J4-Pad22)
- J4 pad 23: Net-(J4-Pad23) -> unconnected-(J4-Pad23)
- J4 pad 25: Net-(J4-Pad25) -> unconnected-(J4-Pad25)
- J4 pad 3: Net-(J4-Pad3) -> unconnected-(J4-Pad3)
- J4 pad 30: Net-(J4-Pad30) -> unconnected-(J4-Pad30)
- J4 pad 31: Net-(J4-Pad31) -> unconnected-(J4-Pad31)
- J4 pad 32: Net-(J4-Pad32) -> unconnected-(J4-Pad32)
- J4 pad 33: Net-(J4-Pad33) -> unconnected-(J4-Pad33)
- J4 pad 44: Net-(J4-Pad44) -> unconnected-(J4-Pad44)
- J4 pad 45: Net-(J4-Pad45) -> unconnected-(J4-Pad45)
- J4 pad 46: Net-(J4-Pad46) -> unconnected-(J4-Pad46)
- J4 pad 47: Net-(J4-Pad47) -> unconnected-(J4-Pad47)
- J4 pad 49: Net-(J4-Pad49) -> unconnected-(J4-Pad49)
- J4 pad 5: Net-(J4-Pad5) -> unconnected-(J4-Pad5)
- J4 pad 51: Net-(J4-Pad51) -> unconnected-(J4-Pad51)
- J4 pad 7: Net-(J4-Pad7) -> unconnected-(J4-Pad7)
- U4 pad 11: Net-(U4-Pad11) -> unconnected-(U4-Pad11)
- U4 pad 12: Net-(U4-Pad12) -> unconnected-(U4-Pad12)
- U4 pad 13: Net-(U4-Pad13) -> unconnected-(U4-Pad13)
- U4 pad 14: Net-(U4-Pad14) -> unconnected-(U4-Pad14)
- U4 pad 16: Net-(U4-Pad16) -> unconnected-(U4-Pad16)
- U4 pad 17: Net-(U4-Pad17) -> unconnected-(U4-Pad17)
- U4 pad 18: Net-(U4-Pad18) -> unconnected-(U4-Pad18)
- U4 pad 19: Net-(U4-Pad19) -> unconnected-(U4-Pad19)
- U4 pad 20: Net-(U4-Pad20) -> unconnected-(U4-Pad20)
- U4 pad 21: Net-(U4-Pad21) -> unconnected-(U4-Pad21)
- U4 pad 34: Net-(U4-Pad34) -> unconnected-(U4-Pad34)
Routing:
- net 3V3_PCI: track 66.4 -> 62.2 mm, vias 12 -> 10
- net unconnected-(C33-Pad1): track 0.00 -> 2.18 mm, vias 0 -> 1
- net unconnected-(C35-Pad1): track 0.00 -> 1.96 mm, vias 0 -> 1
- net unconnected-(C33-Pad2): track 0.00 -> 1.78 mm, vias 0 -> 1
- net GND: track 29.9 -> 28.1 mm, vias 78 -> 77
Other:
- net class Default removed
- board text added: "REV_00"
- board text removed: "REV_01"
